File: PiZeroW-carrier/USB.sch (KiCad schematic (older format))
At the start: 5 parts, among them P1 USB_OTG

Commit message: localize and update USB Micro footprint to match datasheet.  Add more datasheets
Parts:
- P1: footprint Connect:USB_Micro-B -> lib_fp:USB_Micro-B
Changed lines of the file:
@@
 F 0 "P1" H 3400 2190 50  0000 C CNN
 F 1 "USB_OTG" H 3075 2515 50  0000 C CNN
-F 2 "Connect:USB_Micro-B" V 3025 2215 50  0001 C CNN
+F 2 "lib_fp:USB_Micro-B" V 3025 2215 50  0001 C CNN
 F 3 "" V 3025 2215 50  0000 C CNN
 	1    3075 2315

Commit message: netlist update and read into pcb
Parts:
- P1: symbol USB_OTG -> USB_OTG-RESCUE-PiZeroW-carrier
Changed lines of the file:
@@
 EESchema Schematic File Version 2
+LIBS:PiZeroW-carrier-rescue
 LIBS:power
 LIBS:device
@@
 $EndDescr
 $Comp
-L USB_OTG P1
+L USB_OTG-RESCUE-PiZeroW-carrier P1
 U 1 1 5A26AF59
 P 3075 2315
@@
 $EndComp
 $Comp
-L GND #PWR14
+L GND #PWR012
 U 1 1 5A26AFAD
 P 3275 2870
-F 0 "#PWR14" H 3275 2620 50  0001 C CNN
+F 0 "#PWR012" H 3275 2620 50  0001 C CNN
 F 1 "GND" H 3275 2720 50  0000 C CNN
 F 2 "" H 3275 2870 50  0000 C CNN
@@
 $EndComp
 $Comp
-L GND #PWR15
+L GND #PWR013
 U 1 1 5A26AFD2
 P 3655 2415
-F 0 "#PWR15" H 3655 2165 50  0001 C CNN
+F 0 "#PWR013" H 3655 2165 50  0001 C CNN
 F 1 "GND" H 3655 2265 50  0000 C CNN
 F 2 "" H 3655 2415 50  0000 C CNN
@@
 $EndComp
 $Comp
-L GND #PWR13
+L GND #PWR014
 U 1 1 5A26AFE7
 P 3175 3170
-F 0 "#PWR13" H 3175 2920 50  0001 C CNN
+F 0 "#PWR014" H 3175 2920 50  0001 C CNN
 F 1 "GND" H 3175 3020 50  0000 C CNN
 F 2 "" H 3175 3170 50  0000 C CNN
@@
 	2905 2795 2905 3550
 $Comp
-L +5V #PWR12
+L +5V #PWR015
 U 1 1 5A26BAF9
 P 2490 2325
-F 0 "#PWR12" H 2490 2175 50  0001 C CNN
+F 0 "#PWR015" H 2490 2175 50  0001 C CNN
 F 1 "+5V" H 2490 2465 50  0000 C CNN
 F 2 "" H 2490 2325 50  0000 C CNN

Commit message: Complete Pizero Layout
Finnished pi zero led PCB board
Parts:
- W1, W2: footprint SMD_Packages:1Pin -> Pin_Headers:Pin_Header_Straight_1x01_Pitch1.00mm
Changed lines of the file:
@@
 F 0 "W1" H 2250 2865 50  0000 C CNN
 F 1 "D-" H 2315 3015 50  0000 C CNN
-F 2 "SMD_Packages:1Pin" H 2515 2815 50  0001 C CNN
+F 2 "Pin_Headers:Pin_Header_Straight_1x01_Pitch1.00mm" H 2515 2815 50  0001 C CNN
 F 3 "" H 2515 2815 50  0000 C CNN
 	1    2315 2815
@@
 F 0 "W2" H 2440 2870 50  0000 C CNN
 F 1 "D+" H 2505 3015 50  0000 C CNN
-F 2 "SMD_Packages:1Pin" H 2705 2815 50  0001 C CNN
+F 2 "Pin_Headers:Pin_Header_Straight_1x01_Pitch1.00mm" H 2705 2815 50  0001 C CNN
 F 3 "" H 2705 2815 50  0000 C CNN
 	1    2505 2815
