File: PiZeroW-carrier/power.sch (KiCad schematic (older format))
At the start: 7 parts, among them CON1 BARREL_JACK, SW1 SW_PUSH, U1 BA50BC0WFP-E2CT, U2 BA06CC0WFP-E2CT

Commit message: load symbol for LDOs
Parts:
- U1, U2: footprint smd-semi:TO-252-5 -> lib_fp:TO-252-5
Changed lines of the file:
@@
 LIBS:contrib
 LIBS:valves
-LIBS:PiZeroW-carrier-cache
-LIBS:raspberrrypi_hat-cache
+LIBS:ba06cc0wfp-e2ct
 EELAYER 25 0
 EELAYER END
@@
 F 0 "U2" H 8615 2345 50  0000 C CNN
 F 1 "BA06CC0WFP-E2CT" H 8765 2795 50  0000 C CNN
-F 2 "smd-semi:TO-252-5" H 8765 2695 50  0000 C CIN
+F 2 "lib_fp:TO-252-5" H 8765 2695 50  0000 C CIN
 F 3 "" H 8765 2595 50  0000 C CNN
 	1    8765 2595
@@
 F 0 "U1" H 4480 2375 50  0000 C CNN
 F 1 "BA50BC0WFP-E2CT" H 4630 2825 50  0000 C CNN
-F 2 "smd-semi:TO-252-5" H 4630 2725 50  0000 C CIN
+F 2 "lib_fp:TO-252-5" H 4630 2725 50  0000 C CIN
 F 3 "" H 4630 2625 50  0000 C CNN
 	1    4630 2625

Commit message: localize and update USB Micro footprint to match datasheet.  Add more datasheets
Parts:
- added D6: D_Schottky, Diodes_SMD:D_SMA_Handsoldering, symbol D_Schottky
Connections:
- net +5V: now also D6.1 (K); no longer U1.4 (VOUT)
- new net: D6.2 (A), U1.4 (VOUT)
Changed lines of the file:
@@
 Text HLabel 3495 2730 0    60   Input ~ 0
 PiDisable
-Text HLabel 5190 2215 0    60   Input ~ 0
+Text HLabel 5190 1915 2    60   Input ~ 0
 +5V
 Text HLabel 3880 2300 0    60   Input ~ 0
@@
 Wire Wire Line
 	5870 4840 5870 4670
+$Comp
+L D_Schottky D6
+U 1 1 5A293905
+P 5190 2065
+F 0 "D6" H 5190 2165 50  0000 C CNN
+F 1 "D_Schottky" H 5190 1965 50  0000 C CNN
+F 2 "Diodes_SMD:D_SMA_Handsoldering" H 5190 2065 50  0001 C CNN
+F 3 "https://www.digikey.ca/product-detail/en/diodes-incorporated/B130-13-F/B130-FDICT-ND/815318" H 5190 2065 50  0001 C CNN
+	1    5190 2065
+	0    1    1    0
+$EndComp
 $EndSCHEMATC

Commit message: netlist update and read into pcb
Parts:
- CON1: footprint HerbsParts:DC_Barrel_Jack_2mm_6mm -> Connectors:BARREL_JACK
Changed lines of the file:
@@
 EESchema Schematic File Version 2
+LIBS:PiZeroW-carrier-rescue
 LIBS:power
 LIBS:device
@@
 $EndComp
 $Comp
-L +BATT #PWR9
+L +BATT #PWR01
 U 1 1 5A254432
 P 8015 2240
-F 0 "#PWR9" H 8015 2090 50  0001 C CNN
+F 0 "#PWR01" H 8015 2090 50  0001 C CNN
 F 1 "+BATT" H 8015 2380 50  0000 C CNN
 F 2 "" H 8015 2240 50  0000 C CNN
@@
 	7630 2695 7630 2210
 $Comp
-L GND #PWR10
+L GND #PWR02
 U 1 1 5A25448E
 P 8765 2985
-F 0 "#PWR10" H 8765 2735 50  0001 C CNN
+F 0 "#PWR02" H 8765 2735 50  0001 C CNN
 F 1 "GND" H 8765 2835 50  0000 C CNN
 F 2 "" H 8765 2985 50  0000 C CNN
@@
 $EndComp
 $Comp
-L GND #PWR11
+L GND #PWR03
 U 1 1 5A2544A4
 P 9265 2980
-F 0 "#PWR11" H 9265 2730 50  0001 C CNN
+F 0 "#PWR03" H 9265 2730 50  0001 C CNN
 F 1 "GND" H 9265 2830 50  0000 C CNN
 F 2 "" H 9265 2980 50  0000 C CNN
@@
 $EndComp
 $Comp
-L +BATT #PWR3
+L +BATT #PWR04
 U 1 1 5A257C25
 P 3880 2270
-F 0 "#PWR3" H 3880 2120 50  0001 C CNN
+F 0 "#PWR04" H 3880 2120 50  0001 C CNN
 F 1 "+BATT" H 3880 2410 50  0000 C CNN
 F 2 "" H 3880 2270 50  0000 C CNN
@@
 	3495 2725 4180 2725
 $Comp
-L GND #PWR4
+L GND #PWR05
 U 1 1 5A257C30
 P 4630 3015
-F 0 "#PWR4" H 4630 2765 50  0001 C CNN
+F 0 "#PWR05" H 4630 2765 50  0001 C CNN
 F 1 "GND" H 4630 2865 50  0000 C CNN
 F 2 "" H 4630 3015 50  0000 C CNN
@@
 $EndComp
 $Comp
-L GND #PWR5
+L GND #PWR06
 U 1 1 5A257C36
 P 5130 3010
-F 0 "#PWR5" H 5130 2760 50  0001 C CNN
+F 0 "#PWR06" H 5130 2760 50  0001 C CNN
 F 1 "GND" H 5130 2860 50  0000 C CNN
 F 2 "" H 5130 3010 50  0000 C CNN
@@
 $EndComp
 $Comp
-L +BATT #PWR1
+L +BATT #PWR07
 U 1 1 5A257F41
 P 3495 1405
-F 0 "#PWR1" H 3495 1255 50  0001 C CNN
+F 0 "#PWR07" H 3495 1255 50  0001 C CNN
 F 1 "+BATT" H 3495 1545 50  0000 C CNN
 F 2 "" H 3495 1405 50  0000 C CNN
@@
 $EndComp
 $Comp
-L GND #PWR2
+L GND #PWR08
 U 1 1 5A2583C3
 P 3495 3440
-F 0 "#PWR2" H 3495 3190 50  0001 C CNN
+F 0 "#PWR08" H 3495 3190 50  0001 C CNN
 F 1 "GND" H 3495 3290 50  0000 C CNN
 F 2 "" H 3495 3440 50  0000 C CNN
@@
 	3495 3345 3495 3440
 $Comp
-L +BATT #PWR8
+L +BATT #PWR09
 U 1 1 5A268E4D
 P 7630 1810
-F 0 "#PWR8" H 7630 1660 50  0001 C CNN
+F 0 "#PWR09" H 7630 1660 50  0001 C CNN
 F 1 "+BATT" H 7630 1950 50  0000 C CNN
 F 2 "" H 7630 1810 50  0000 C CNN
@@
 F 0 "CON1" H 5405 5190 50  0000 C CNN
 F 1 "BARREL_JACK" H 5405 4740 50  0000 C CNN
-F 2 "HerbsParts:DC_Barrel_Jack_2mm_6mm" H 5405 4940 50  0001 C CNN
+F 2 "Connectors:BARREL_JACK" H 5405 4940 50  0001 C CNN
 F 3 "" H 5405 4940 50  0000 C CNN
 	1    5405 4940
@@
 $EndComp
 $Comp
-L GND #PWR7
+L GND #PWR010
 U 1 1 5A26A00C
 P 5870 5135
-F 0 "#PWR7" H 5870 4885 50  0001 C CNN
+F 0 "#PWR010" H 5870 4885 50  0001 C CNN
 F 1 "GND" H 5870 4985 50  0000 C CNN
 F 2 "" H 5870 5135 50  0000 C CNN
@@
 Connection ~ 5870 5040
 $Comp
-L +BATT #PWR6
+L +BATT #PWR011
 U 1 1 5A26A0AC
 P 5870 4670
-F 0 "#PWR6" H 5870 4520 50  0001 C CNN
+F 0 "#PWR011" H 5870 4520 50  0001 C CNN
 F 1 "+BATT" H 5870 4810 50  0000 C CNN
 F 2 "" H 5870 4670 50  0000 C CNN

Commit message: Before Trace fix of LED AND PIDISABLE
Push before tracing fix of LEDEnable and PIDisable
Connections:
- wire segments 25 -> 28
Changed lines of the file:
@@
 Wire Wire Line
 	9330 2545 9330 2185
-Text HLabel 7985 2975 0    60   Input ~ 0
-LEDEnable
 Text HLabel 9330 2185 0    60   Input ~ 0
 +6V
@@
 Wire Wire Line
 	5190 2575 5190 2215
-Text HLabel 3495 2730 0    60   Input ~ 0
+Text HLabel 3400 2700 0    60   Input ~ 0
 PiDisable
 Text HLabel 5190 1915 2    60   Input ~ 0
@@
 	0    1    1    0
 $EndComp
+Wire Wire Line
+	3401 2699 3452 2699
+Wire Wire Line
+	3452 2699 3452 2725
+Wire Wire Line
+	3452 2725 3494 2725
+Text HLabel 7985 2975 0    60   Input ~ 0
+LEDEnable
 $EndSCHEMATC

Commit message: cleanup some routes that the autorouter must have created
Changed lines of the file:
@@
 Wire Wire Line
 	5190 2575 5190 2215
-Text HLabel 3400 2700 0    60   Input ~ 0
+Text HLabel 3500 2725 0    60   Input ~ 0
 PiDisable
 Text HLabel 5190 1915 2    60   Input ~ 0
@@
 Wire Wire Line
 	3452 2725 3494 2725
-Text HLabel 7985 2975 0    60   Input ~ 0
+Text HLabel 7985 2975 0    60   Output ~ 0
 LEDEnable
 $EndSCHEMATC

Commit message: fix PiDisable/LEDEnable.  Need to connect them on the root sheet. Extra-duh
Connections:
- wire segments 28 -> 25
Changed lines of the file:
@@
 Wire Wire Line
 	5190 2575 5190 2215
-Text HLabel 3500 2725 0    60   Input ~ 0
+Text HLabel 3495 2725 0    60   Input ~ 0
 PiDisable
 Text HLabel 5190 1915 2    60   Input ~ 0
@@
 	0    1    1    0
 $EndComp
-Wire Wire Line
-	3401 2699 3452 2699
-Wire Wire Line
-	3452 2699 3452 2725
-Wire Wire Line
-	3452 2725 3494 2725
-Text HLabel 7985 2975 0    60   Output ~ 0
+Text HLabel 7985 2975 0    60   Input ~ 0
 LEDEnable
 $EndSCHEMATC
