File: PiZeroW-carrier/raspberrypi-gpio-40pin.sch (KiCad schematic (older format))
At the start: 5 parts, among them J1 PI40HAT

Commit message: fix PiDisable/LEDEnable.  Need to connect them on the root sheet. Extra-duh
Changed lines of the file:
@@
 	1    0    0    -1
 $EndComp
-Text HLabel 1495 2750 0    60   Output ~ 0
+Text HLabel 1495 2750 0    60   Input ~ 0
 LEDEnable
 $EndSCHEMATC
