File: PiZeroW-carrier/backup.kicad_pcb (KiCad board)
At the start: 2 copper layers, 65 x 30 mm, 26 parts, among them CON1 BARREL_JACK, J1 PI40HAT, P1 USB_OTG, SW1 SW_PUSH, U1 BA50BC0WFP-E2CT, U2 BA06CC0WFP-E2CT

Commit message: Push of (Hopefully) Finnished board
Need  silkscreen stuff
Parts:
- moved R7 32.2 mm to (162.6, 96.3), turned to 270 degrees
- moved R6 24.1 mm to (155.4, 96.3), turned to 270 degrees
- moved SW1 18.1 mm to (142.8, 104.5), turned to 270 degrees
- moved R4 18.1 mm to (149.5, 96.3), turned to 270 degrees
- moved R1 17.7 mm to (140.9, 96.3), turned to 270 degrees
- moved R8 14.3 mm to (144.4, 96.2), turned to 270 degrees
Routing:
- net Net-(D4-Pad4): track 39.0 -> 7.74 mm
- net Net-(R1-Pad2): track 42.0 -> 11.0 mm, vias 3 -> 1
- net +BATT: track 78.9 -> 53.3 mm, vias 4 -> 0
- net Net-(D3-Pad4): track 29.9 -> 7.83 mm
- net Net-(R2-Pad1): track 30.5 -> 11.0 mm, vias 1 -> 0
- net /Leds/+6V: track 0.00 -> 18.2 mm
- net Net-(D1-Pad4): track 21.4 -> 7.88 mm
- net Net-(D5-Pad4): track 14.7 -> 8.32 mm
