File: PiZeroW-carrier/PiZeroW-carrier.kicad_pcb (KiCad board)
At the start: 2 copper layers, 65 x 30 mm, 26 parts, among them CON1 BARREL_JACK, J1 PI40HAT, P1 USB_OTG, SW1 SW_PUSH, U1 BA50BC0WFP-E2CT, U2 BA06CC0WFP-E2CT

Commit message: PCb Now with PIDisable and 6V Connection.
Featuring a PCB With proper PIDisable and 6V Connections
Connections:
- D6 pad 1: /Power/+5V -> (no net)
- J1 pad 1: /raspberrypi-gpio-40pin/P3V3_HAT -> (no net)
- J1 pad 10: Net-(J1-Pad10) -> (no net)
- J1 pad 12: Net-(J1-Pad12) -> (no net)
- J1 pad 13: /Power/PiDisable -> /Power/PIDisable
- J1 pad 15: Net-(J1-Pad15) -> (no net)
- J1 pad 16: Net-(J1-Pad16) -> (no net)
- J1 pad 17: Net-(J1-Pad17) -> (no net)
- J1 pad 18: Net-(J1-Pad18) -> (no net)
- J1 pad 19: Net-(J1-Pad19) -> (no net)
- J1 pad 21: Net-(J1-Pad21) -> (no net)
- J1 pad 22: Net-(J1-Pad22) -> (no net)
- J1 pad 23: Net-(J1-Pad23) -> (no net)
- J1 pad 24: Net-(J1-Pad24) -> (no net)
- J1 pad 26: Net-(J1-Pad26) -> (no net)
- J1 pad 27: /raspberrypi-gpio-40pin/SDA -> (no net)
- J1 pad 28: /raspberrypi-gpio-40pin/SCL -> (no net)
- J1 pad 29: Net-(J1-Pad29) -> (no net)
- J1 pad 3: Net-(J1-Pad3) -> (no net)
- J1 pad 31: Net-(J1-Pad31) -> (no net)
- J1 pad 32: Net-(J1-Pad32) -> (no net)
- J1 pad 33: Net-(J1-Pad33) -> (no net)
- J1 pad 35: Net-(J1-Pad35) -> (no net)
- J1 pad 36: Net-(J1-Pad36) -> (no net)
- J1 pad 37: Net-(J1-Pad37) -> (no net)
- J1 pad 38: Net-(J1-Pad38) -> (no net)
- J1 pad 40: Net-(J1-Pad40) -> (no net)
- J1 pad 5: Net-(J1-Pad5) -> (no net)
- J1 pad 7: Net-(J1-Pad7) -> (no net)
- J1 pad 8: Net-(J1-Pad8) -> (no net)
- R1 pad 2: Net-(R1-Pad2) -> (no net)
- R12 pad 1: +5V -> (no net)
- R2 pad 1: Net-(R2-Pad1) -> /Power/PIDisable
- SW1 pad 1: Net-(R2-Pad1) -> /Power/PIDisable
- SW1 pad 2: Net-(R1-Pad2) -> Net-(SW1-Pad2)
- U1 pad 1: Net-(R2-Pad1) -> /Power/PIDisable
- U2 pad 4: /Power/+6V -> /Leds/+6V
Routing:
- net Net-(SW1-Pad2): track 0.00 -> 42.0 mm, vias 0 -> 3
- net Net-(R1-Pad2): track 42.0 -> 0.00 mm, vias 3 -> 0
- net Net-(R2-Pad1): track 30.5 -> 0.00 mm, vias 1 -> 0
- net /Power/PIDisable: track 0.00 -> 30.5 mm, vias 0 -> 1
- net /Leds/+6V: track 0.00 -> 14.3 mm

Commit message: SILKS START.
Start of the silks mdude
Parts:
- moved D6 11.2 mm to (136.6, 107.3), turned to 0 degrees
- moved R2 10.0 mm to (144.4, 100.8)
- moved R3 9.68 mm to (144.5, 107.2), turned to 180 degrees
- moved R11 7.77 mm to (144.4, 102.9)
Routing:
- net GND: track 16.2 -> 127.1 mm, vias 0 -> 4
- net /Power/PIDisable: track 30.5 -> 134.4 mm, vias 1 -> 7
- net /Power/LEDEnable: track 5.73 -> 88.8 mm, vias 1 -> 2
- net /Leds/+6V: track 14.3 -> 46.9 mm, vias 0 -> 3
- net +BATT: track 78.9 -> 89.2 mm, vias 4 -> 6
- net Net-(D6-Pad2): track 16.0 -> 21.4 mm
- net Net-(P1-Pad4): track 23.7 -> 28.9 mm
- net /raspberrypi-gpio-40pin/P5V_HAT: track 0.13 -> 2.54 mm
Other:
- board text added: "BARREL_JACK/PLUG"
- board text added: "BATTERY CONNECTION FOR RESET BUTTON"
- board text added: "I CANT REMEMBER WHAT THIS IS CALLED"
- board text added: "LED 1"
- board text added: "LED 1 RESISTOR"
- board text added: "LED 2"
- board text added: "LED 2 RESISTOR"
- board text added: "LED 3"
- board text added: "LED 3 RESISTOR"
- board text added: "LED 4"
- board text added: "LED 4 RESISTOR"
- board text added: "LED ENABLE RESISTOR"
- board text added: "PIDISABLE RESISTOR"
- board text added: "RESET BUTTON PIDISABLE"
- board text added: "USB"

Commit message: Most(Possibly All Silks)
Most of ( or maybe all silks????? added to the board!.
Other:
- board text added: "SCHOTTKY"
Changed lines of the file:
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@@
     (area 109.424999 79.424999 174.575001 109.575001)
     (thickness 1.6)
-    (drawings 28)
+    (drawings 29)
     (tracks 289)
     (zones 0)
@@
     (descr "DC Barrel Jack")
     (tags "Power Jack")
-    (fp_text reference CON1 (at -8.45 5.75 360) (layer F.SilkS)
+    (fp_text reference CON1 (at -8.45 5.75 180) (layer F.SilkS) hide
       (effects (font (size 1 1) (thickness 0.15)))
     )
@@
     (tags "Diode SMA (DO-214AC) Handsoldering")
     (attr smd)
-    (fp_text reference D6 (at 0 2.5) (layer B.SilkS)
-      (effects (font (size 1 1) (thickness 0.15)) (justify mirror))
-    )
-    (fp_text value D_Schottky (at 0 -2.6) (layer B.Fab)
+    (fp_text reference D6 (at 0 2.5) (layer B.SilkS) hide
+      (effects (font (size 1 1) (thickness 0.15)) (justify mirror))
+    )
+    (fp_text value D_Schottky (at 0 -2.6) (layer B.Fab) hide
       (effects (font (size 1 1) (thickness 0.15)) (justify mirror))
     )
@@
       (effects (font (size 1 1) (thickness 0.15)) (justify mirror))
     )
-    (fp_text value 150 (at 0 -1.9) (layer B.Fab)
+    (fp_text value 150 (at 0 -1.9) (layer B.Fab) hide
       (effects (font (size 1 1) (thickness 0.15)) (justify mirror))
     )
@@
       (effects (font (size 1 1) (thickness 0.15)) (justify mirror))
     )
-    (fp_text value 10k (at 0 -1.75 180) (layer B.Fab)
+    (fp_text value 10k (at 0 -1.75 180) (layer B.Fab) hide
       (effects (font (size 1 1) (thickness 0.15)) (justify mirror))
     )
@@
       (effects (font (size 1 1) (thickness 0.15)) (justify mirror))
     )
-    (fp_text value 150 (at 0 -1.9 180) (layer B.Fab)
+    (fp_text value 150 (at 0 -1.9 180) (layer B.Fab) hide
       (effects (font (size 1 1) (thickness 0.15)) (justify mirror))
     )
@@
       (effects (font (size 1 1) (thickness 0.15)) (justify mirror))
     )
-    (fp_text value 150 (at 0 -1.9 180) (layer B.Fab)
+    (fp_text value 150 (at 0 -1.9 180) (layer B.Fab) hide
       (effects (font (size 1 1) (thickness 0.15)) (justify mirror))
     )
@@
       (effects (font (size 1 1) (thickness 0.15)) (justify mirror))
     )
-    (fp_text value 150 (at 0 -1.9 180) (layer B.Fab)
+    (fp_text value 150 (at 0 -1.9 180) (layer B.Fab) hide
       (effects (font (size 1 1) (thickness 0.15)) (justify mirror))
     )
@@
       (effects (font (size 1 1) (thickness 0.15)) (justify mirror))
     )
-    (fp_text value 150 (at 0 -1.9 180) (layer B.Fab)
+    (fp_text value 150 (at 0 -1.9 180) (layer B.Fab) hide
       (effects (font (size 1 1) (thickness 0.15)) (justify mirror))
     )
@@
       (effects (font (size 1 1) (thickness 0.15)) (justify mirror))
     )
-    (fp_text value DNP (at 0 -1.75 180) (layer B.Fab)
+    (fp_text value DNP (at 0 -1.75 180) (layer B.Fab) hide
       (effects (font (size 1 1) (thickness 0.15)) (justify mirror))
     )
@@
       (clearance 1.6))
   )
+  (gr_text SCHOTTKY (at 136.3472 105.0544) (layer B.SilkS)
+    (effects (font (size 0.5 0.5) (thickness 0.125)) (justify mirror))
+  )
   (gr_text "PIDISABLE RESISTOR" (at 144.3228 99.7712) (layer B.SilkS)
-    (effects (font (size 0.127 0.127) (thickness 0.01) italic))
-  )
-  (gr_text "BATTERY CONNECTION FOR RESET BUTTON" (at 125.603 85.725) (layer B.SilkS)
-    (effects (font (size 0.25 0.25) (thickness 0.0625) italic))
+    (effects (font (size 0.127 0.127) (thickness 0.01) italic) (justify mirror))
+  )
+  (gr_text "BATTERY CONNECTION FOR RESET BUTTON" (at 125.5776 85.979) (layer B.SilkS)
+    (effects (font (size 0.25 0.25) (thickness 0.0625) italic) (justify mirror))
   )
   (gr_text "LED ENABLE RESISTOR" (at 144.6276 108.458) (layer B.SilkS)
-    (effects (font (size 0.3 0.3) (thickness 0.075) italic))
+    (effects (font (size 0.3 0.3) (thickness 0.075) italic) (justify mirror))
   )
   (gr_text "I CANT REMEMBER WHAT THIS IS CALLED" (at 165.2016 108.7628) (layer B.SilkS)
-    (effects (font (size 0.25 0.25) (thickness 0.0625) italic))
+    (effects (font (size 0.25 0.25) (thickness 0.0625) italic) (justify mirror))
   )
   (gr_text "I CANT REMEMBER WHAT THIS IS CALLED" (at 165.2016 108.7628) (layer F.SilkS)
@@
   )
   (gr_text "LED 4 RESISTOR" (at 127.9906 104.4956 270) (layer B.SilkS)
-    (effects (font (size 0.2 0.25) (thickness 0.05) italic))
+    (effects (font (size 0.2 0.25) (thickness 0.05) italic) (justify mirror))
   )
   (gr_text "LED 3 RESISTOR" (at 128.0922 99.7458 270) (layer B.SilkS)
-    (effects (font (size 0.2 0.25) (thickness 0.05) italic))
+    (effects (font (size 0.2 0.25) (thickness 0.05) italic) (justify mirror))
   )
   (gr_text "LED 2 RESISTOR\n" (at 128.0922 95.123 270) (layer B.SilkS)
-    (effects (font (size 0.2 0.25) (thickness 0.05) italic))
+    (effects (font (size 0.2 0.25) (thickness 0.05) italic) (justify mirror))
   )
   (gr_text "LED 1 RESISTOR" (at 128.0922 90.2462 270) (layer B.SilkS)
-    (effects (font (size 0.2 0.25) (thickness 0.05) italic))
+    (effects (font (size 0.2 0.25) (thickness 0.05) italic) (justify mirror))
   )
   (gr_text "LED 4" (at 165.5826 89.3318) (layer F.SilkS)
@@
   )
   (gr_text USB (at 172.9486 95.9104 270) (layer B.SilkS)
-    (effects (font (size 1 1) (thickness 0.25) italic))
+    (effects (font (size 1 1) (thickness 0.25) italic) (justify mirror))
   )
   (gr_line (start 171.5 109.5) (end 170.95 109.5) (angle 90) (layer Edge.Cuts) (width 0.15))

Commit message: FINISHED BOARD
Finished Board Yeet
Other:
- board text added: "1"
- board text added: "4627"
- board text added: "BY Sam Sheppard 2018"
- board text added: "DM"
- board text added: "DP"
- board text added: "LDO BA50"
- board text added: "LDO BAO6"
- board text added: "RESET"
- board text removed: "I CANT REMEMBER WHAT THIS IS CALLED"
Changed lines of the file:
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@@
     (area 109.424999 79.424999 174.575001 109.575001)
     (thickness 1.6)
-    (drawings 29)
+    (drawings 38)
     (tracks 289)
     (zones 0)
@@
   )
   (setup
-    (last_trace_width 0.254)
+    (last_trace_width 0.6)
     (user_trace_width 0.6)
     (trace_clearance 0.254)
@@
       (effects (font (size 0.762 0.762) (thickness 0.1016)))
     )
-    (fp_text value LED_QBLP679E (at 0 -3.2 270) (layer F.SilkS)
+    (fp_text value LED_QBLP679E (at 0 -3.2 270) (layer F.SilkS) hide
       (effects (font (size 0.762 0.762) (thickness 0.1016)))
     )
@@
       (effects (font (size 0.762 0.762) (thickness 0.1016)))
     )
-    (fp_text value LED_QBLP679E (at 0 -3.2 270) (layer F.SilkS)
+    (fp_text value LED_QBLP679E (at 0 -3.2 270) (layer F.SilkS) hide
       (effects (font (size 0.762 0.762) (thickness 0.1016)))
     )
@@
       (effects (font (size 0.762 0.762) (thickness 0.1016)))
     )
-    (fp_text value LED_QBLP679E (at 0 -3.2 270) (layer F.SilkS)
+    (fp_text value LED_QBLP679E (at 0 -3.2 270) (layer F.SilkS) hide
       (effects (font (size 0.762 0.762) (thickness 0.1016)))
     )
@@
       (effects (font (size 1 1) (thickness 0.15)))
     )
-    (fp_text value SW_PUSH (at 0 3.75 180) (layer F.Fab)
+    (fp_text value SW_PUSH (at 0 3.75 180) (layer F.Fab) hide
       (effects (font (size 1 1) (thickness 0.15)))
     )
@@
       (effects (font (size 1 1) (thickness 0.15)))
     )
-    (fp_text value PI40HAT (at 1.27 50.59 90) (layer F.Fab)
+    (fp_text value PI40HAT (at 1.27 50.59 90) (layer F.Fab) hide
       (effects (font (size 1 1) (thickness 0.15)))
     )
@@
       (effects (font (size 1 1) (thickness 0.15)) (justify mirror))
     )
-    (fp_text value D- (at 0 -1.56 270) (layer B.Fab)
+    (fp_text value D- (at 0 -1.56 270) (layer B.Fab) hide
       (effects (font (size 1 1) (thickness 0.15)) (justify mirror))
     )
@@
       (effects (font (size 1 1) (thickness 0.15)) (justify mirror))
     )
-    (fp_text value D+ (at 0 -1.56 270) (layer B.Fab)
+    (fp_text value D+ (at 0 -1.56 270) (layer B.Fab) hide
       (effects (font (size 1 1) (thickness 0.15)) (justify mirror))
     )
@@
       (effects (font (size 1 1) (thickness 0.15)))
     )
-    (fp_text value Hole_3mm_PTH (at 0 -2.7) (layer F.Fab)
+    (fp_text value Hole_3mm_PTH (at 0 -2.7) (layer F.Fab) hide
       (effects (font (size 1 1) (thickness 0.15)))
     )
@@
       (effects (font (size 1 1) (thickness 0.15)))
     )
-    (fp_text value Hole_3mm_PTH (at 0 -2.7) (layer F.Fab)
+    (fp_text value Hole_3mm_PTH (at 0 -2.7) (layer F.Fab) hide
       (effects (font (size 1 1) (thickness 0.15)))
     )
@@
       (clearance 1.6))
   )
+  (gr_text 1 (at 167.4876 85.6488) (layer F.SilkS)
+    (effects (font (size 0.2 0.2) (thickness 0.05) italic))
+  )
+  (gr_text 1 (at 160.5788 85.471) (layer F.SilkS)
+    (effects (font (size 0.2 0.2) (thickness 0.05) italic))
+  )
+  (gr_text 1 (at 154.1526 85.471) (layer F.SilkS)
+    (effects (font (size 0.2 0.2) (thickness 0.05) italic))
+  )
+  (gr_text 1 (at 148.2852 85.3948) (layer F.SilkS)
+    (effects (font (size 0.2 0.2) (thickness 0.05) italic))
+  )
+  (gr_text "4627 " (at 123.5964 103.6574) (layer F.SilkS)
+    (effects (font (size 1 1) (thickness 0.25)))
+  )
+  (gr_text "BY Sam Sheppard 2018" (at 123.5456 102.2096) (layer F.SilkS)
+    (effects (font (size 0.5 0.5) (thickness 0.125)))
+  )
+  (gr_text RESET (at 163.068 97.1042 90) (layer F.SilkS)
+    (effects (font (size 0.25 0.25) (thickness 0.0625) italic))
+  )
+  (gr_text DP (at 169.926 102.9716) (layer F.Cu)
+    (effects (font (size 0.5 0.5) (thickness 0.125)))
+  )
+  (gr_text DM (at 173.4312 103.0986) (layer F.Cu)
+    (effects (font (size 0.5 0.5) (thickness 0.125)))
+  )
   (gr_text SCHOTTKY (at 136.3472 105.0544) (layer B.SilkS)
     (effects (font (size 0.5 0.5) (thickness 0.125)) (justify mirror))
@@
     (effects (font (size 0.3 0.3) (thickness 0.075) italic) (justify mirror))
   )
-  (gr_text "I CANT REMEMBER WHAT THIS IS CALLED" (at 165.2016 108.7628) (layer B.SilkS)
+  (gr_text "LDO BA50\n" (at 165.2016 108.7628) (layer B.SilkS)
     (effects (font (size 0.25 0.25) (thickness 0.0625) italic) (justify mirror))
   )
-  (gr_text "I CANT REMEMBER WHAT THIS IS CALLED" (at 165.2016 108.7628) (layer F.SilkS)
+  (gr_text "LDO BAO6\n\n\n " (at 165.2016 109.3978) (layer F.SilkS)
     (effects (font (size 0.25 0.25) (thickness 0.0625) italic))
   )
